File: Hardware/RadioLab.brd (EAGLE design)
At the start: 80 x 40 mm, 54 parts, among them Q1 16MHz, U1 USB, U2 V_REG_LDOSMD, U3 NRF24L01SMD, U6 ATMEGA32U4-AU, X3 16MHz

Commit message: Updated SCH and BRD
Parts:
- removed C20: 10uF, SparkFun:EIA3216
- removed LED5, LED7: Yellow, led:1206
- removed SW1: (no value), special:EDG-05
- removed U6: ATMEGA32U4-AU, IC:TQFP44
- added C17: 1.5pF, resistor:C0402
- added LED3, LED4: Yellow, led:SML0603
- added R9: 10k, resistor:R0402
- added RA1: RESISTOR_ARRAY_8PIN, SpaceDIY_IC:CRA12E
- added S1: A6S-5104-H, SpaceDIY_connectors:A6S-5104-H
- added S2: Reset, Testing:TACTILE_SWITCH_TALL
- added SV1: USB, daspilker:FCI-10103594-0001LF
- C18: value 1.5pF -> 10uF; device resistor:C0402 -> SparkFun:EIA3216
- LED1, LED2: device led:1206 -> led:SML0603
- R7, R8: device SparkFun:C0402 -> resistor:R0402
- U1: value USB -> ATMEGA32U4-AU; device daspilker:FCI-10103594-0001LF -> adafruit:TQFP44
- moved U1 21.2 mm to (34.4, 15.5), turned to 270 degrees
- moved C18 9.67 mm to (46.9, 26.0), flipped to the top
- moved R1 8.94 mm to (13.0, 3.00)
- moved R2 8.94 mm to (25.0, 3.00)
- moved R6 5.33 mm to (39.8, 26.9)
- moved C8 3.32 mm to (43.2, 22.9), turned to 0 degrees
- moved LED1 1.80 mm to (31.4, 2.40)
- moved R5 1.77 mm to (28.2, 3.50), turned to 90 degrees
- moved C2 0.98 mm to (36.1, 2.60)
- moved C1 0.92 mm to (22.1, 15.8)
- moved LED2 0.82 mm to (39.8, 28.2)
- moved C12 0.63 mm to (38.4, 33.7)
- moved C11 0.60 mm to (34.6, 23.4)
- moved R7 0.54 mm to (43.6, 25.2)
- moved C7 0.51 mm to (43.3, 25.5), turned to 270 degrees
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- renumbered J$2 to ANT
Connections:
- net 3.3V: now also C18.A; no longer C20.A
- net A0: now also U1.36; no longer U6.36
- net A1: now also U1.37; no longer U6.37
- net A2: now also U1.38; no longer U6.38
- net A3: now also U1.39; no longer U6.39
- net A4: now also U1.40; no longer U6.40
- net A5: now also U1.41; no longer U6.41
- net ANT: now also C17.1; no longer C18.1
- net AREF: now also U1.42; no longer U6.42
- net D+: now also U1.4; no longer U6.4
- net D-: now also U1.3; no longer U6.3
- net D0: now also RA1.1, S1.5, U1.20; no longer SW1.10, U6.20
- net D1: now also RA1.2, S1.4, U1.21; no longer SW1.9, U6.21
- net D10: now also U1.30; no longer U6.30
- net D11: now also U1.12; no longer U6.12
- net D12: now also U1.26; no longer U6.26
- net D13: now also U1.32; no longer U6.32
- net D14: now also U1.11; no longer U6.11
- net D15: now also U1.9; no longer U6.9
- net D16: now also U1.10; no longer U6.10
- net D17/PB0/RXLED1: now also U1.8; no longer U6.8
- net D2: now also RA1.3, S1.3, U1.19; no longer SW1.8, U6.19
- net D3: now also RA1.4, S1.2, U1.18; no longer SW1.7, U6.18
- net D4: now also RA1.5, S1.1, U1.25; no longer SW1.6, U6.25
- net D5: now also U1.31; no longer U6.31
- net D6: now also U1.27; no longer U6.27
- net D7: now also U1.1; no longer U6.1
- net D8: now also U1.28; no longer U6.28
- net D9: now also U1.29; no longer U6.29
- net GND: now also C18.C, RA1.8, S2.A2, SV1.5, U1.15, U1.23, U1.33, U1.35, U1.43; no longer C20.C, U6.15, U6.23, U6.33, U6.35, U6.43, U6.5
- net N$15: now also LED4.C; no longer LED7.C
- net N$16: now also LED3.C; no longer LED5.C
- net N$2: now also SV1.3; no longer U1.3
- net N$3: now also U1.17; no longer U6.17
- net N$4: now also SV1.2; no longer U1.2
- net N$7: now also U1.16; no longer U6.16
- net PD5/TXLED1: now also U1.22; no longer U6.22
- net RST: now also R9.2, S2.B2, U1.13; no longer U6.13
- net TANT: now also C17.2; no longer C18.2
- net UCAP1: now also U1.6; no longer U6.6
- net VBUS: now also SV1.1; no longer U1.1
- net VCC: now also LED3.A, LED4.A, R9.1, S1.10, S1.6, S1.7, S1.8, S1.9, U1.14, U1.2, U1.24, U1.34, U1.44, U1.7; no longer LED5.A, LED7.A, SW1.1, SW1.2, SW1.3, SW1.4, SW1.5, U6.14, U6.2, U6.24, U6.34, U6.44, U6.7
Routing:
- net A1: track 39.0 -> 101.2 mm, vias 1 -> 2
- net A0: track 44.8 -> 106.1 mm, vias 1 -> 4
- net A2: track 31.4 -> 92.1 mm, vias 1 -> 2
- net A3: track 28.7 -> 89.0 mm, vias 1 -> 3
- net VCC: track 185.2 -> 132.9 mm, vias 8 -> 11
- net D11: track 37.5 -> 80.9 mm
- net D8: track 9.66 -> 47.4 mm, vias 1 -> 3
- net D5: track 26.0 -> 63.3 mm, vias 0 -> 1
- net D6: track 39.2 -> 70.7 mm
- net D9: track 34.6 -> 61.7 mm
- net D4: track 35.9 -> 55.3 mm, vias 1 -> 5
- net D10: track 32.8 -> 52.1 mm
- net N$3: track 10.3 -> 29.0 mm, vias 1 -> 3
- net D17/PB0/RXLED1: track 15.8 -> 33.6 mm
- net N$7: track 7.84 -> 23.1 mm
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Other:
- outline, holes or cut-outs redrawn

Commit message: Global updates
Parts:
- C1, C10, C11, C12, C13, C14, C15, C16, C17, C2, C3, C4, C5, C6, C7, C8, C9: device resistor:C0402 -> SpaceDIY_passive_components:0402
- L1, L2, L3: device SparkFun:C0402 -> SpaceDIY_passive_components:0402
- LED1, LED2, LED3, LED4: device led:SML0603 -> SpaceDIY_passive_components:LED0402
- R1, R2, R3, R4, R5, R6, R7, R8, R9: device resistor:R0402 -> SpaceDIY_passive_components:0402
- moved C15 1.70 mm to (30.9, 30.1)
- moved C16 1.20 mm to (33.1, 30.1)
- moved C6 1.10 mm to (38.5, 23.9)
- moved C14 1.10 mm to (43.1, 22.7)
- moved R6 0.85 mm to (39.9, 26.1), turned to 0 degrees
- moved L2 0.80 mm to (35.2, 30.1)
- moved C13 0.50 mm to (28.0, 27.1)
- moved R7 0.40 mm to (43.6, 24.8)
- moved C7 0.16 mm to (43.4, 25.6), turned to 90 degrees
- moved L3 0.10 mm to (37.4, 30.1)
- moved LED2 0.09 mm to (39.9, 28.1), turned to 0 degrees
Connections:
- net GND: now also C7.2; no longer C7.1
- net VCC: now also C7.1; no longer C7.2
Routing:
- net GND: track 2.31 -> 0.20 mm, vias 25 -> 26
- net D13: track 35.5 -> 33.8 mm
- net N$10: track 6.02 -> 7.69 mm
- net N$9: track 1.34 -> 2.18 mm
- net N$12: track 3.01 -> 3.78 mm
- net N$13: track 4.39 -> 5.09 mm
- net N$5: track 10.3 -> 10.8 mm
Other:
- board text added: "0"
- board text added: "1"
- board text added: "ANT"
- board text added: "Channel"
- board text added: "Mode"
- board text added: "Power"
- board text added: "Reset"
- board text added: "Rx"
- board text added: "Tx"
