File: Hardware/RadioLab.sch (EAGLE design)
At the start: 54 parts, among them Q1 16MHz, U1 USB, U2 V_REG_LDOSMD, U3 NRF24L01SMD, U6 ATMEGA32U4-AU, X3 16MHz

Commit message: Updated SCH and BRD
Parts:
- removed C20: 10uF, SparkFun:CAP_POL1206
- removed LED5, LED7: Yellow, led:LEDSMT1206
- removed SW1: (no value), special:SW_DIP-5
- removed U6: ATMEGA32U4-AU, IC:ATMEGA32U4-AU
- added C17: 1.5pF, resistor:C-USC0402
- added LED3, LED4: Yellow, led:LEDSML0603
- added R9: 10k, resistor:R-US_R0402
- added RA1: RESISTOR_ARRAY_8PIN, SpaceDIY_IC:RESISTOR_ARRAY_8PIN
- added S1: A6S-5104-H, SpaceDIY_connectors:A6S-5104-H
- added S2: Reset, Testing:SWITCH-MOMENTARY-2SMD-4
- added SV1: USB, daspilker:USB-RECEPTABLE
- C18: value 1.5pF -> 10uF; device resistor:C-USC0402 -> SparkFun:CAP_POL1206
- LED1, LED2: device led:LEDSMT1206 -> led:LEDSML0603
- R7, R8: device SparkFun:RESISTOR0402 -> resistor:R-US_R0402
- U1: value USB -> ATMEGA32U4-AU; device daspilker:USB-RECEPTABLE -> adafruit:ATMEGA32U4-AU
- renumbered J$2 to ANT
Connections:
- net 3.3V: now also C18.+; no longer C20.+
- net A0: now also U1.PF7(ADC7(TDI); no longer U6.PF7(ADC7/TDI)
- net A1: now also U1.PF6(ADC6/TDO); no longer U6.PF6(ADC6/TDO)
- net A2: now also U1.PF5(ADC5/TMS); no longer U6.PF5(ADC5/TMS)
- net A3: now also U1.PF4(ADC4/TCK); no longer U6.PF4(ADC4/TCK)
- net A4: now also U1.PF1(ADC1); no longer U6.PF1(ADC1)
- net A5: now also U1.PF0(ADC0); no longer U6.PF0(ADC0)
- net ANT: now also C17.1; no longer C18.1
- net AREF: now also U1.AREF; no longer U6.AREF
- net D+: now also U1.D+; no longer U6.D+
- net D-: now also U1.D-; no longer U6.D-
- net D0: now also RA1.1, S1.5, U1.PD2(INT2/RXD1); no longer SW1.10, U6.PD2(RXD1/INT2)
- net D1: now also RA1.2, S1.4, U1.PD3(INT3/TXD1); no longer SW1.9, U6.PD3(TXD1/INT3)
- net D10: now also U1.PB6(OC1B/OC4B/ADC13); no longer U6.PB6(PCINT6/OC1B/OC4B/ADC13)
- net D11: now also U1.PB7(OC0A/OC1C/RTS); no longer U6.PB7(PCINT7/OC0A/OC1C/!RTS)
- net D12: now also U1.PD6(T1/ADC9/!OC4D); no longer U6.PD6(T1/ADC9/!OC4D)
- net D13: now also U1.PC7(ICP3/CLK0/OC4A); no longer U6.PC7(ICP3/CLK0/OC4A)
- net D14: now also U1.PB3(PDO/MISO); no longer U6.PB3(PD0/PCINT3/MISO)
- net D15: now also U1.PB1(SCK); no longer U6.PB1(PCINT1/SCLK)
- net D16: now also U1.PB2(PDI/MOSI); no longer U6.PB2(PDI/PCINT2/MOSI)
- net D17/PB0/RXLED1: now also U1.PB0(SS); no longer U6.PB0(SS/PCINT0)
- net D2: now also RA1.3, S1.3, U1.PD1(INT1/SDA); no longer SW1.8, U6.PD1(SDA/INT1)
- net D3: now also RA1.4, S1.2, U1.PD0(INT0/OC0B/SCL); no longer SW1.7, U6.PD0(OC0B/SCL/INT0)
- net D4: now also RA1.5, S1.1, U1.PD4(ICP1/ADC8); no longer SW1.6, U6.PD4(ICP1/ADC8)
- net D5: now also U1.PC6(OC3A/!OC4A); no longer U6.PC6(OC3A/!OC4A)
- net D6: now also U1.PD7(OC4D/ADC10/T0); no longer U6.PD7(T0/OC4D/ADC10)
- net D7: now also U1.PE6(INT.6/AIN0); no longer U6.PE6(INT.6/AIN0)
- net D8: now also U1.PB4(ADC11); no longer U6.PB4(PCINT4/ADC11)
- net D9: now also U1.PB5(OC1A/ADC12/!OC4B); no longer U6.PB5(PCINT5/OC1A/ADC12/!OC4B)
- net GND: now also C18.-, RA1.8, S2.1, SV1.GND, U1.GND1, U1.GND2, U1.GND3, U1.PE2(!HWB), U1.UGND; no longer C20.-, U6.GND@1, U6.GND@2, U6.GND@3, U6.GND@4, U6.PE2(!HWB), U6.UGND
- net N$15: now also LED4.C; no longer LED7.C
- net N$16: now also LED3.C; no longer LED5.C
- net N$2: now also SV1.D+; no longer U1.D+
- net N$3: now also U1.XTAL1; no longer U6.XTAL1
- net N$4: now also SV1.D-; no longer U1.D-
- net N$7: now also U1.XTAL2; no longer U6.XTAL2
- net PD5/TXLED1: now also U1.PD5(XCK/CTS); no longer U6.PD5(XCLK1/!CTS)
- net RST: now also R9.2, S2.2, U1./RESET; no longer U6.!RESET
- net TANT: now also C17.2; no longer C18.2
- net UCAP1: now also U1.UCAP; no longer U6.UCAP
- net VBUS: now also SV1.VCC; no longer U1.VCC
- net VCC: now also LED3.A, LED4.A, R9.1, S1.10, S1.6, S1.7, S1.8, S1.9, U1.AVCC, U1.AVCC1, U1.UVCC, U1.VBUS, U1.VCC, U1.VCC1; no longer LED5.A, LED7.A, SW1.1, SW1.2, SW1.3, SW1.4, SW1.5, U6.AVCC@1, U6.AVCC@2, U6.UVCC, U6.VBUS, U6.VCC@1, U6.VCC@2
Other:
- moved on the sheet: C1, C2, C3, R1, R2, R3, R4, SV2, X3

Commit message: Global updates
Parts:
- C1, C10, C11, C12, C13, C14, C15, C16, C17, C2, C3, C4, C5, C6, C7, C8, C9: device resistor:C-USC0402 -> SpaceDIY_passive_components:C0402
- L1, L2, L3: device SparkFun:INDUCTOR0402 -> SpaceDIY_passive_components:L0402
- LED1, LED2, LED3, LED4: device led:LEDSML0603 -> SpaceDIY_passive_components:LED0402
- R1, R2, R3, R4, R5, R6, R7, R8, R9: device resistor:R-US_R0402 -> SpaceDIY_passive_components:R0402
Connections:
- net GND: now also C7.2; no longer C7.1
- net VCC: now also C7.1; no longer C7.2
Other:
- moved on the sheet: C7, LED1, LED2, LED3, LED4
